File: hardware/powermeter_supply/powermeter.brd (EAGLE design)
At the start: 97.1 x 61.9 mm, 24 parts, among them J1 AUDIO_JACK_3.5MM_KIT, X2 MSTBA2

Commit message: Update finalisation
Parts:
- removed C1: 470µF, rcl:E5-8,5
- removed C2: 47µF, rcl:E2,5-5
- removed JP1: (no value), pinhead:1X02
- removed R6, R7, R8, R9: 10k, rcl:0204/7
- removed SJ1: (no value), jumper:SJ
- removed U$3: MINI-UPS-S, mini-ups:MINI-UPS-S
- moved R1 36.6 mm to (25.4, 8.26)
- moved R2 36.5 mm to (21.6, 8.26)
- moved U$2 12.1 mm to (76.2, 30.5)
- moved R3 11.7 mm to (12.7, 52.4)
- moved U1 11.4 mm to (20.3, 29.8), turned to 90 degrees
- moved C4 10.6 mm to (24.4, 54.9)
- moved R5 9.10 mm to (16.5, 52.4)
- moved R4 8.80 mm to (20.3, 52.4)
- moved J1 8.35 mm to (33.7, 58.4)
- moved U$1 1.91 mm to (51.4, 24.4)
- moved X2 1.91 mm to (51.4, 59.7)
Connections:
- removed net BAT: R8.2, R9.1, U1.IO34
- removed net N$5: R7.2, SJ1.1, U$2.+V, U$3.VIN
- removed net N$6: JP1.2, R9.2, U$3.BAT
- removed net VIN: R6.2, R7.1, U1.IO32
- net +3V3: no longer C2.+
- net CURRENT: now also U1.IO32; no longer U1.IO33
- net GND: now also U1.IO4; no longer C1.-, C2.-, JP1.1, R6.1, R8.1, U$3.P$1, U$3.P$3, U$3.P$4
- net VCC: now also U$2.+V; no longer C1.+, SJ1.2, U$3.OUT
- net VOLTAGE: now also U1.IO34; no longer U1.IO36
Routing:
- net BAT: track 74.2 -> 0.00 mm
- net N$1: track 84.1 -> 36.3 mm
- net VIN: track 39.8 -> 0.00 mm
- net VCC: track 127.5 -> 94.3 mm
- net N$5: track 29.4 -> 0.00 mm
- net VOLTAGE: track 33.6 -> 7.62 mm
- net +3V3: track 54.7 -> 32.8 mm
- net CURRENT: track 41.8 -> 20.3 mm
- net N$6: track 16.2 -> 0.00 mm
- net N$4: track 40.7 -> 31.9 mm
- net N$2: track 20.7 -> 28.8 mm
- net N$3: track 27.8 -> 21.9 mm
- net GND: track 5.22 -> 4.36 mm
Other:
- outline, holes or cut-outs redrawn
