File: hardware/powermeter_supply/powermeter.sch (EAGLE design)
At the start: 24 parts, among them J1 AUDIO_JACK_3.5MM_KIT, X2 MSTBA2

Commit message: Update finalisation
Parts:
- removed C1: 470µF, rcl:CPOL-EUE5-8.5
- removed C2: 47µF, rcl:CPOL-EUE2.5-5
- removed JP1: (no value), pinhead:PINHD-1X2
- removed R6, R7, R8, R9: 10k, rcl:R-EU_0204/7
- removed SJ1: (no value), jumper:SJ
- removed U$3: MINI-UPS-S, mini-ups:MINI-UPS-S
Connections:
- removed net BAT: R8.2, R9.1, U1.GPIO34/ADC1-6
- removed net N$5: R7.2, SJ1.1, U$2.+V, U$3.VIN
- removed net N$6: JP1.2, R9.2, U$3.BAT
- removed net VIN: R6.2, R7.1, U1.GPIO32/ADC1-4
- net +3V3: no longer C2.+
- net CURRENT: now also U1.GPIO32/ADC1-4; no longer U1.GPIO33/ADC1-5
- net GND: now also U1.GPIO4; no longer C1.-, C2.-, JP1.1, R6.1, R8.1, U$3.GND
- net VCC: now also U$2.+V; no longer C1.+, SJ1.2, U$3.OUT
- net VOLTAGE: now also U1.GPIO34/ADC1-6; no longer U1.GPIO36/ADC1-0
Other:
- moved on the sheet: H1, H2, H3, H4
